Commit message: Updated for Gazebo integration

File: hexapod_description/urdf/hexapod_body.xacro (robot description, xacro)
@@ -2,4 +2,10 @@
 <robot name="hexapod" xmlns:xacro="https://www.ros.org/wiki/xacro">
 	<xacro:include filename="$(find hexapod_description)/urdf/links_joints_macro.xacro" />
+	<!-- Used for fixing robot to Gazebo 'base_link' -->
+		<link name="world"/>
+ 		<joint name="fixed" type="fixed">
+  			<parent link="world"/>
+   			<child link="base_link"/>
+ 		 </joint>
 		<m_link name="base_link"
 				origin_xyz="0 0 0" origin_rpy="0 0 0"
@@ -9,5 +15,5 @@
 					 effort="1000.0" lower="-1.5708" upper="1.5708" velocity="0.5"
 			 		 origin_xyz="0.072981 0.109608 0" origin_rpy="0 0 -0.7854"
-					 parent="base_link" child="leg1_coxa" />
+					 parent="base_link" child="leg1_coxa" damping="0.7"/>
 			<m_link name="leg1_coxa"
 					origin_xyz="0 0 0.021" origin_rpy="0 0 0"
@@ -16,5 +22,5 @@
 				 effort="1000.0" lower="-1.5708" upper="1.5708" velocity="0.5"
 				 origin_xyz="0 0.047868 0.021" origin_rpy="0 0 0"
-				 parent="leg1_coxa" child="leg1_femur" />
+				 parent="leg1_coxa" child="leg1_femur" damping="0.7"/>
 				<m_link name="leg1_femur"
 						origin_xyz="0 0.0385 0" origin_rpy="0 3.14159 0"
@@ -23,5 +29,5 @@
 					 effort="1000.0" lower="-1.5708" upper="1.5708" velocity="0.5"
 					 origin_xyz="0 0.077 0" origin_rpy="0 0 0"
-					 parent="leg1_femur" child="leg1_tibia" />
+					 parent="leg1_femur" child="leg1_tibia" damping="0.7"/>
 					<m_link name="leg1_tibia"
 							origin_xyz="0 0 0" origin_rpy="3.14159 0 1.5708"
@@ -31,5 +37,5 @@
 					 effort="1000.0" lower="-1.5708" upper="1.5708" velocity="0.5"
 			 		 origin_xyz="-0.072981 0.109608 0" origin_rpy="0 0 0.7854"
-					 parent="base_link" child="leg2_coxa" />
+					 parent="base_link" child="leg2_coxa" damping="0.7"/>
 			<m_link name="leg2_coxa"
 					origin_xyz="0 0 0.021" origin_rpy="0 0 0"
@@ -38,5 +44,5 @@
 						 effort="1000.0" lower="-1.5708" upper="1.5708" velocity="0.5"
 						 origin_xyz="0 0.047868 0.021" origin_rpy="0 0 0"
-						 parent="leg2_coxa" child="leg2_femur" />
+						 parent="leg2_coxa" child="leg2_femur" damping="0.7"/>
 				<m_link name="leg2_femur"
 						origin_xyz="0 0.0385 0" origin_rpy="0 3.14159 0"
@@ -45,5 +51,5 @@
 					 effort="1000.0" lower="-1.5708" upper="1.5708" velocity="0.5"
 					 origin_xyz="0 0.077 0" origin_rpy="0 0 0"
-					 parent="leg2_femur" child="leg2_tibia" />
+					 parent="leg2_femur" child="leg2_tibia" damping="0.7"/>
 					<m_link name="leg2_tibia"
 							origin_xyz="0 0 0" origin_rpy="3.14159 0 1.5708"
@@ -53,5 +59,5 @@
 					 effort="1000.0" lower="-1.5708" upper="1.5708" velocity="0.5"
 			 		 origin_xyz="0.09850 0 0" origin_rpy="0 0 -1.5708"
-					 parent="base_link" child="leg3_coxa" />
+					 parent="base_link" child="leg3_coxa" damping="0.7"/>
 			<m_link name="leg3_coxa"
 					origin_xyz="0 0 0.021" origin_rpy="0 0 0"
@@ -60,5 +66,5 @@
 						 effort="1000.0" lower="-1.5708" upper="1.5708" velocity="0.5"
 						 origin_xyz="0 0.047868 0.021" origin_rpy="0 0 0"
-						 parent="leg3_coxa" child="leg3_femur" />
+						 parent="leg3_coxa" child="leg3_femur" damping="0.7"/>
 				<m_link name="leg3_femur"
 						origin_xyz="0 0.0385 0" origin_rpy="0 3.14159 0"
@@ -67,5 +73,5 @@
 					 effort="1000.0" lower="-1.5708" upper="1.5708" velocity="0.5"
 					 origin_xyz="0 0.077 0" origin_rpy="0 0 0"
-					 parent="leg3_femur" child="leg3_tibia" />
+					 parent="leg3_femur" child="leg3_tibia" damping="0.7"/>
 					<m_link name="leg3_tibia"
 							origin_xyz="0 0 0" origin_rpy="3.14159 0 1.5708"
@@ -75,5 +81,5 @@
 					 effort="1000.0" lower="-1.5708" upper="1.5708" velocity="0.5"
 			 		 origin_xyz="-0.09850 0 0" origin_rpy="0 0 1.5708"
-					 parent="base_link" child="leg4_coxa" />
+					 parent="base_link" child="leg4_coxa" damping="0.7"/>
 			<m_link name="leg4_coxa"
 					origin_xyz="0 0 0.021" origin_rpy="0 0 0"
@@ -82,5 +88,5 @@
 				 effort="1000.0" lower="-1.5708" upper="1.5708" velocity="0.5"
 				 origin_xyz="0 0.047868 0.021" origin_rpy="0 0 0"
-				 parent="leg4_coxa" child="leg4_femur" />
+				 parent="leg4_coxa" child="leg4_femur" damping="0.7"/>
 				<m_link name="leg4_femur"
 						origin_xyz="0 0.0385 0" origin_rpy="0 3.14159 0"
@@ -89,5 +95,5 @@
 					 effort="1000.0" lower="-1.5708" upper="1.5708" velocity="0.5"
 					 origin_xyz="0 0.077 0" origin_rpy="0 0 0"
-					 parent="leg4_femur" child="leg4_tibia" />
+					 parent="leg4_femur" child="leg4_tibia" damping="0.7"/>
 					<m_link name="leg4_tibia"
 							origin_xyz="0 0 0" origin_rpy="3.14159 0 1.5708"
@@ -97,5 +103,5 @@
 					 effort="1000.0" lower="-1.5708" upper="1.5708" velocity="0.5"
 			 		 origin_xyz="0.072981 -0.109608 0" origin_rpy="0 0 -2.3562"
-					 parent="base_link" child="leg5_coxa" />
+					 parent="base_link" child="leg5_coxa" damping="0.7"/>
 			<m_link name="leg5_coxa"
 					origin_xyz="0 0 0.021" origin_rpy="0 0 0"
@@ -104,5 +110,5 @@
 						 effort="1000.0" lower="-1.5708" upper="1.5708" velocity="0.5"
 						 origin_xyz="0 0.047868 0.021" origin_rpy="0 0 0"
-						 parent="leg5_coxa" child="leg5_femur" />
+						 parent="leg5_coxa" child="leg5_femur" damping="0.7"/>
 				<m_link name="leg5_femur"
 						origin_xyz="0 0.0385 0" origin_rpy="0 3.14159 0"
@@ -111,5 +117,5 @@
 					 effort="1000.0" lower="-1.5708" upper="1.5708" velocity="0.5"
 					 origin_xyz="0 0.077 0" origin_rpy="0 0 0"
-					 parent="leg5_femur" child="leg5_tibia" />
+					 parent="leg5_femur" child="leg5_tibia" damping="0.7"/>
 					<m_link name="leg5_tibia"
 							origin_xyz="0 0 0" origin_rpy="3.14159 0 1.5708"
@@ -119,5 +125,5 @@
 					 effort="1000.0" lower="-1.5708" upper="1.5708" velocity="0.5"
 			 		 origin_xyz="-0.072981 -0.109608 0" origin_rpy="0 0 2.3562"
-					 parent="base_link" child="leg6_coxa" />
+					 parent="base_link" child="leg6_coxa" damping="0.7"/>
 			<m_link name="leg6_coxa"
 					origin_xyz="0 0 0.021" origin_rpy="0 0 0"
@@ -126,5 +132,5 @@
 						 effort="1000.0" lower="-1.5708" upper="1.5708" velocity="0.5"
 						 origin_xyz="0 0.047868 0.021" origin_rpy="0 0 0"
-						 parent="leg6_coxa" child="leg6_femur" />
+						 parent="leg6_coxa" child="leg6_femur" damping="0.7"/>
 				<m_link name="leg6_femur"
 						origin_xyz="0 0.0385 0" origin_rpy="0 3.14159 0"
@@ -133,5 +139,5 @@
 					 effort="1000.0" lower="-1.5708" upper="1.5708" velocity="0.5"
 					 origin_xyz="0 0.077 0" origin_rpy="0 0 0"
-					 parent="leg6_femur" child="leg6_tibia" />
+					 parent="leg6_femur" child="leg6_tibia" damping="0.7"/>
 					<m_link name="leg6_tibia"
 							origin_xyz="0 0 0" origin_rpy="3.14159 0 1.5708"

File: hexapod_description/urdf/links_joints_macro.xacro (robot description, xacro)
@@ -1,6 +1,17 @@
 <?xml version="1.0"?>
 <robot xmlns:xacro="https://www.ros.org/wiki/xacro">
+  <!-- Import all Gazebo-customization elements, including Gazebo colors -->
+  <xacro:include filename="$(find hexapod_description)/urdf/hexapod.gazebo" />
+  <!-- Import Rviz colors -->
+  <xacro:include filename="$(find hexapod_description)/urdf/materials.xacro" />
+  <xacro:property name="mass" value="1" /> <!-- arbitrary value for mass -->
 	<xacro:macro name="m_link" params="name origin_xyz origin_rpy mesh_file mesh_scale">
 		<link name="${name}">
+			<collision>
+				<origin xyz="${origin_xyz}" rpy="${origin_rpy}" />
+				<geometry>
+					<mesh filename="${mesh_file}" scale="${mesh_scale}" />
+				</geometry>
+			</collision>
 			<visual>
 				<origin xyz="${origin_xyz}" rpy="${origin_rpy}" />
@@ -8,8 +19,14 @@
 					<mesh filename="${mesh_file}" scale="${mesh_scale}" />
 				</geometry>
+				<material name="red" />
 			</visual>
+			<inertial>
+      			<origin xyz="${origin_xyz}" rpy="${origin_rpy}"/>
+      			<mass value="${mass}"/>
+      			<inertia ixx="1.0" ixy="0.0" ixz="0.0" iyy="0.5" iyz="0.0" izz="1.0" />
+    		</inertial>
 		</link>
 	</xacro:macro>
-	<xacro:macro name="m_joint" params="name type axis_xyz effort lower upper velocity origin_xyz origin_rpy parent child" >
+	<xacro:macro name="m_joint" params="name type axis_xyz effort lower upper velocity origin_xyz origin_rpy parent child damping" >
 		<joint name="${name}" type="${type}">
 			<axis xyz="${axis_xyz}" />
@@ -18,4 +35,5 @@
 			<parent link="${parent}" />
 			<child link="${child}" />
+			<dynamics damping="${damping}"/>
 		</joint>
 	</xacro:macro>

Commit message: Updated inertial values

File: hexapod_description/urdf/hexapod_body.xacro (robot description, xacro)
@@ -8,6 +8,6 @@
    			<child link="base_link"/>
  		 </joint>
-		<m_link name="base_link"
-				origin_xyz="0 0 0" origin_rpy="0 0 0"
+		<m_base_link name="base_link"
+				origin_xyz="0 0 0" origin_rpy="0 0 0" inertia_origin_xyz="-0.00000000611 0.000002 0.021504"
 				mesh_file="package://hexapod_description/meshes/base_link.stl" mesh_scale="0.001 0.001 0.001" />
 		<!-- LEG 1 (North East) -->
@@ -16,6 +16,6 @@
 			 		 origin_xyz="0.072981 0.109608 0" origin_rpy="0 0 -0.7854"
 					 parent="base_link" child="leg1_coxa" damping="0.7"/>
-			<m_link name="leg1_coxa"
-					origin_xyz="0 0 0.021" origin_rpy="0 0 0"
+			<m_coxa_link name="leg1_coxa"
+					origin_xyz="0 0 0.021" origin_rpy="0 0 0" inertia_origin_xyz="0.00006 0.023937 0.00006"
 					mesh_file="package://hexapod_description/meshes/leg_coxa.stl" mesh_scale="0.001 0.001 0.001" />
 				<m_joint name="leg1_coxa__leg1_femur" type="revolute" axis_xyz="1 0 0"
@@ -23,6 +23,7 @@
 				 origin_xyz="0 0.047868 0.021" origin_rpy="0 0 0"
 				 parent="leg1_coxa" child="leg1_femur" damping="0.7"/>
-				<m_link name="leg1_femur"
+				<m_femur_link name="leg1_femur"
 						origin_xyz="0 0.0385 0" origin_rpy="0 3.14159 0"
+						inertia_origin_xyz="0.000216 -0.0000003648 -0.00000000863"
 						mesh_file="package://hexapod_description/meshes/leg_femur.stl" mesh_scale="0.001 0.001 0.001" />
 					<m_joint name="leg1_femur__leg1_tibia" type="revolute" axis_xyz="1 0 0"
@@ -30,6 +31,7 @@
 					 origin_xyz="0 0.077 0" origin_rpy="0 0 0"
 					 parent="leg1_femur" child="leg1_tibia" damping="0.7"/>
-					<m_link name="leg1_tibia"
+					<m_tibia_link name="leg1_tibia"
 							origin_xyz="0 0 0" origin_rpy="3.14159 0 1.5708"
+							inertia_origin_xyz="0.083874 0.000095 0.046294"
 							mesh_file="package://hexapod_description/meshes/leg_tibia.stl" mesh_scale="0.001 0.001 0.001" />
 		<!-- LEG 2 (North West) -->
@@ -38,6 +40,6 @@
 			 		 origin_xyz="-0.072981 0.109608 0" origin_rpy="0 0 0.7854"
 					 parent="base_link" child="leg2_coxa" damping="0.7"/>
-			<m_link name="leg2_coxa"
-					origin_xyz="0 0 0.021" origin_rpy="0 0 0"
+			<m_coxa_link name="leg2_coxa"
+					origin_xyz="0 0 0.021" origin_rpy="0 0 0" inertia_origin_xyz="0.00006 0.023937 0.00006"
 					mesh_file="package://hexapod_description/meshes/leg_coxa.stl" mesh_scale="0.001 0.001 0.001" />
 				<m_joint name="leg2_coxa__leg2_femur" type="revolute" axis_xyz="1 0 0"
@@ -45,6 +47,7 @@
 						 origin_xyz="0 0.047868 0.021" origin_rpy="0 0 0"
 						 parent="leg2_coxa" child="leg2_femur" damping="0.7"/>
-				<m_link name="leg2_femur"
+				<m_femur_link name="leg2_femur"
 						origin_xyz="0 0.0385 0" origin_rpy="0 3.14159 0"
+						inertia_origin_xyz="0.000216 -0.0000003648 -0.00000000863"
 						mesh_file="package://hexapod_description/meshes/leg_femur.stl" mesh_scale="0.001 0.001 0.001" />
 					<m_joint name="leg2_femur__leg2_tibia" type="revolute" axis_xyz="1 0 0"
@@ -52,6 +55,7 @@
 					 origin_xyz="0 0.077 0" origin_rpy="0 0 0"
 					 parent="leg2_femur" child="leg2_tibia" damping="0.7"/>
-					<m_link name="leg2_tibia"
+					<m_tibia_link name="leg2_tibia"
 							origin_xyz="0 0 0" origin_rpy="3.14159 0 1.5708"
+							inertia_origin_xyz="0.083874 0.000095 0.046294"
 							mesh_file="package://hexapod_description/meshes/leg_tibia.stl" mesh_scale="0.001 0.001 0.001" />
 		<!-- LEG 3 (East) -->
@@ -60,5 +64,5 @@
 			 		 origin_xyz="0.09850 0 0" origin_rpy="0 0 -1.5708"
 					 parent="base_link" child="leg3_coxa" damping="0.7"/>
-			<m_link name="leg3_coxa"
+			<m_coxa_link name="leg3_coxa" inertia_origin_xyz="0.00006 0.023937 0.00006"
 					origin_xyz="0 0 0.021" origin_rpy="0 0 0"
 					mesh_file="package://hexapod_description/meshes/leg_coxa.stl" mesh_scale="0.001 0.001 0.001" />
@@ -67,6 +71,7 @@
 						 origin_xyz="0 0.047868 0.021" origin_rpy="0 0 0"
 						 parent="leg3_coxa" child="leg3_femur" damping="0.7"/>
-				<m_link name="leg3_femur"
+				<m_femur_link name="leg3_femur"
 						origin_xyz="0 0.0385 0" origin_rpy="0 3.14159 0"
+						inertia_origin_xyz="0.000216 -0.0000003648 -0.00000000863"
 						mesh_file="package://hexapod_description/meshes/leg_femur.stl" mesh_scale="0.001 0.001 0.001" />
 					<m_joint name="leg3_femur__leg3_tibia" type="revolute" axis_xyz="1 0 0"
@@ -74,6 +79,7 @@
 					 origin_xyz="0 0.077 0" origin_rpy="0 0 0"
 					 parent="leg3_femur" child="leg3_tibia" damping="0.7"/>
-					<m_link name="leg3_tibia"
+					<m_tibia_link name="leg3_tibia"
 							origin_xyz="0 0 0" origin_rpy="3.14159 0 1.5708"
+							inertia_origin_xyz="0.083874 0.000095 0.046294"
 							mesh_file="package://hexapod_description/meshes/leg_tibia.stl" mesh_scale="0.001 0.001 0.001" />
 		<!-- LEG 4 (West) -->
@@ -82,6 +88,6 @@
 			 		 origin_xyz="-0.09850 0 0" origin_rpy="0 0 1.5708"
 					 parent="base_link" child="leg4_coxa" damping="0.7"/>
-			<m_link name="leg4_coxa"
-					origin_xyz="0 0 0.021" origin_rpy="0 0 0"
+			<m_coxa_link name="leg4_coxa"
+					origin_xyz="0 0 0.021" origin_rpy="0 0 0" inertia_origin_xyz="0.00006 0.023937 0.00006"
 					mesh_file="package://hexapod_description/meshes/leg_coxa.stl" mesh_scale="0.001 0.001 0.001" />
 				<m_joint name="leg4_coxa__leg4_femur" type="revolute" axis_xyz="1 0 0"
@@ -89,6 +95,7 @@
 				 origin_xyz="0 0.047868 0.021" origin_rpy="0 0 0"
 				 parent="leg4_coxa" child="leg4_femur" damping="0.7"/>
-				<m_link name="leg4_femur"
+				<m_femur_link name="leg4_femur"
 						origin_xyz="0 0.0385 0" origin_rpy="0 3.14159 0"
+						inertia_origin_xyz="0.000216 -0.0000003648 -0.00000000863"
 						mesh_file="package://hexapod_description/meshes/leg_femur.stl" mesh_scale="0.001 0.001 0.001" />
 					<m_joint name="leg4_femur__leg4_tibia" type="revolute" axis_xyz="1 0 0"
@@ -96,6 +103,7 @@
 					 origin_xyz="0 0.077 0" origin_rpy="0 0 0"
 					 parent="leg4_femur" child="leg4_tibia" damping="0.7"/>
-					<m_link name="leg4_tibia"
+					<m_tibia_link name="leg4_tibia"
 							origin_xyz="0 0 0" origin_rpy="3.14159 0 1.5708"
+							inertia_origin_xyz="0.083874 0.000095 0.046294"
 							mesh_file="package://hexapod_description/meshes/leg_tibia.stl" mesh_scale="0.001 0.001 0.001" />
 		<!-- LEG 5 (South East) -->
@@ -104,6 +112,6 @@
 			 		 origin_xyz="0.072981 -0.109608 0" origin_rpy="0 0 -2.3562"
 					 parent="base_link" child="leg5_coxa" damping="0.7"/>
-			<m_link name="leg5_coxa"
-					origin_xyz="0 0 0.021" origin_rpy="0 0 0"
+			<m_coxa_link name="leg5_coxa"
+					origin_xyz="0 0 0.021" origin_rpy="0 0 0" inertia_origin_xyz="0.00006 0.023937 0.00006"
 					mesh_file="package://hexapod_description/meshes/leg_coxa.stl" mesh_scale="0.001 0.001 0.001" />
 				<m_joint name="leg5_coxa__leg5_femur" type="revolute" axis_xyz="1 0 0"
@@ -111,6 +119,7 @@
 						 origin_xyz="0 0.047868 0.021" origin_rpy="0 0 0"
 						 parent="leg5_coxa" child="leg5_femur" damping="0.7"/>
-				<m_link name="leg5_femur"
+				<m_femur_link name="leg5_femur"
 						origin_xyz="0 0.0385 0" origin_rpy="0 3.14159 0"
+						inertia_origin_xyz="0.000216 -0.0000003648 -0.00000000863"
 						mesh_file="package://hexapod_description/meshes/leg_femur.stl" mesh_scale="0.001 0.001 0.001" />
 					<m_joint name="leg5_femur__leg5_tibia" type="revolute" axis_xyz="1 0 0"
@@ -118,6 +127,7 @@
 					 origin_xyz="0 0.077 0" origin_rpy="0 0 0"
 					 parent="leg5_femur" child="leg5_tibia" damping="0.7"/>
-					<m_link name="leg5_tibia"
+					<m_tibia_link name="leg5_tibia"
 							origin_xyz="0 0 0" origin_rpy="3.14159 0 1.5708"
+							inertia_origin_xyz="0.083874 0.000095 0.046294"
 							mesh_file="package://hexapod_description/meshes/leg_tibia.stl" mesh_scale="0.001 0.001 0.001" />
 		<!-- LEG 6 (South West) -->
@@ -126,6 +136,6 @@
 			 		 origin_xyz="-0.072981 -0.109608 0" origin_rpy="0 0 2.3562"
 					 parent="base_link" child="leg6_coxa" damping="0.7"/>
-			<m_link name="leg6_coxa"
-					origin_xyz="0 0 0.021" origin_rpy="0 0 0"
+			<m_coxa_link name="leg6_coxa"
+					origin_xyz="0 0 0.021" origin_rpy="0 0 0" inertia_origin_xyz="0.00006 0.023937 0.00006"
 					mesh_file="package://hexapod_description/meshes/leg_coxa.stl" mesh_scale="0.001 0.001 0.001" />
 				<m_joint name="leg6_coxa__leg6_femur" type="revolute" axis_xyz="1 0 0"
@@ -133,6 +143,7 @@
 						 origin_xyz="0 0.047868 0.021" origin_rpy="0 0 0"
 						 parent="leg6_coxa" child="leg6_femur" damping="0.7"/>
-				<m_link name="leg6_femur"
+				<m_femur_link name="leg6_femur"
 						origin_xyz="0 0.0385 0" origin_rpy="0 3.14159 0"
+						inertia_origin_xyz="0.000216 -0.0000003648 -0.00000000863"
 						mesh_file="package://hexapod_description/meshes/leg_femur.stl" mesh_scale="0.001 0.001 0.001" />
 					<m_joint name="leg6_femur__leg6_tibia" type="revolute" axis_xyz="1 0 0"
@@ -140,6 +151,7 @@
 					 origin_xyz="0 0.077 0" origin_rpy="0 0 0"
 					 parent="leg6_femur" child="leg6_tibia" damping="0.7"/>
-					<m_link name="leg6_tibia"
+					<m_tibia_link name="leg6_tibia"
 							origin_xyz="0 0 0" origin_rpy="3.14159 0 1.5708"
+							inertia_origin_xyz="0.083874 0.000095 0.046294"
 							mesh_file="package://hexapod_description/meshes/leg_tibia.stl" mesh_scale="0.001 0.001 0.001" />
 </robot>

File: hexapod_description/urdf/links_joints_macro.xacro (robot description, xacro)
@@ -5,6 +5,5 @@
   <!-- Import Rviz colors -->
   <xacro:include filename="$(find hexapod_description)/urdf/materials.xacro" />
-  <xacro:property name="mass" value="1" /> <!-- arbitrary value for mass -->
-	<xacro:macro name="m_link" params="name origin_xyz origin_rpy mesh_file mesh_scale">
+	<xacro:macro name="m_base_link" params="name origin_xyz origin_rpy inertia_origin_xyz mesh_file mesh_scale">
 		<link name="${name}">
 			<collision>
@@ -22,7 +21,81 @@
 			</visual>
 			<inertial>
-      			<origin xyz="${origin_xyz}" rpy="${origin_rpy}"/>
-      			<mass value="${mass}"/>
-      			<inertia ixx="1.0" ixy="0.0" ixz="0.0" iyy="0.5" iyz="0.0" izz="1.0" />
+      			<origin xyz="${inertia_origin_xyz}" rpy="${origin_rpy}"/>
+      			<mass value="4"/>
+      			<inertia ixx="0.02109" 		   ixy="-0.000000524323" ixz="0.000000000016"
+      					 iyx="-0.000000524323" iyy="0.0144" 		 iyz="0.000003891"
+      					 izx="0.000000000016"  izy="0.000003891" 	 izz="0.0373"/>
+    		</inertial>
+		</link>
+	</xacro:macro>
+	<xacro:macro name="m_coxa_link" params="name origin_xyz origin_rpy inertia_origin_xyz mesh_file mesh_scale">
+		<link name="${name}">
+			<collision>
+				<origin xyz="${origin_xyz}" rpy="${origin_rpy}" />
+				<geometry>
+					<mesh filename="${mesh_file}" scale="${mesh_scale}" />
+				</geometry>
+			</collision>
+			<visual>
+				<origin xyz="${origin_xyz}" rpy="${origin_rpy}" />
+				<geometry>
+					<mesh filename="${mesh_file}" scale="${mesh_scale}" />
+				</geometry>
+				<material name="red" />
+			</visual>
+			<inertial>
+      			<origin xyz="${inertia_origin_xyz}" rpy="${origin_rpy}"/>
+      			<mass value="0.2"/>
+      			<inertia ixx="0.00008176" 	   ixy="-0.000000295397" ixz="0.000000000742"
+      					 iyx="-0.000000295397" iyy="0.0001025" 		 iyz="0.000000293619"
+      					 izx="0.000000000742"  izy="0.000000293619"  izz="0.00008176"/>
+    		</inertial>
+		</link>
+	</xacro:macro>
+	<xacro:macro name="m_femur_link" params="name origin_xyz origin_rpy inertia_origin_xyz mesh_file mesh_scale">
+		<link name="${name}">
+			<collision>
+				<origin xyz="${origin_xyz}" rpy="${origin_rpy}" />
+				<geometry>
+					<mesh filename="${mesh_file}" scale="${mesh_scale}" />
+				</geometry>
+			</collision>
+			<visual>
+				<origin xyz="${origin_xyz}" rpy="${origin_rpy}" />
+				<geometry>
+					<mesh filename="${mesh_file}" scale="${mesh_scale}" />
+				</geometry>
+				<material name="red" />
+			</visual>
+			<inertial>
+      			<origin xyz="${inertia_origin_xyz}" rpy="${origin_rpy}"/>
+      			<mass value="0.7"/>
+      			<inertia ixx="0.0000616" 	   ixy="0.000000004936"  ixz="-0.000000000097"
+      					 iyx="0.000000004936"  iyy="0.0001212" 		 iyz="0.000000357772"
+      					 izx="-0.000000000097" izy="0.000000357772"  izz="0.0006537"/>
+    		</inertial>
+		</link>
+	</xacro:macro>
+	<xacro:macro name="m_tibia_link" params="name origin_xyz origin_rpy inertia_origin_xyz mesh_file mesh_scale">
+		<link name="${name}">
+			<collision>
+				<origin xyz="${origin_xyz}" rpy="${origin_rpy}" />
+				<geometry>
+					<mesh filename="${mesh_file}" scale="${mesh_scale}" />
+				</geometry>
+			</collision>
+			<visual>
+				<origin xyz="${origin_xyz}" rpy="${origin_rpy}" />
+				<geometry>
+					<mesh filename="${mesh_file}" scale="${mesh_scale}" />
+				</geometry>
+				<material name="red" />
+			</visual>
+			<inertial>
+      			<origin xyz="${inertia_origin_xyz}" rpy="${origin_rpy}"/>
+      			<mass value="0.5"/>
+      			<inertia ixx="0.00126"	 	   ixy="0.000003599427"  ixz="-0.0007157"
+      					 iyx="0.000003599427"  iyy="0.001877" 		 iyz="0.000002060961"
+      					 izx="-0.0007157" 	   izy="0.000002060961"  izz="0.0008954"/>
     		</inertial>
 		</link>
