Commit message: Added the new rubber link

File: hexapod_description/urdf/hexapod_body.xacro (robot description, xacro)
@@ -35,4 +35,10 @@
 							inertia_origin_xyz="0.083874 0.000095 0.046294"
 							mesh_file="package://hexapod_description/meshes/leg_tibia.stl" mesh_scale="0.001 0.001 0.001" />
+						<m_joint_fixed name="leg1_tibia__leg1_rubber_tip" type="fixed"
+						 parent="leg1_tibia" child="leg1_rubber_tip" />
+						<m_rubber_tip_link name="leg1_rubber_tip"
+								origin_xyz="0 0.136283 -0.133814" origin_rpy="3.5185838 0 0"
+								inertia_origin_xyz="0.083874 0.000095 0.046294"
+								mesh_file="package://hexapod_description/meshes/leg_rubber_tip.stl" mesh_scale="0.001 0.001 0.001" />
 		<!-- LEG 2 (North West) -->
 			<m_joint name="base_link__leg2_coxa" type="revolute" axis_xyz="0 0 1"
@@ -59,4 +65,10 @@
 							inertia_origin_xyz="0.083874 0.000095 0.046294"
 							mesh_file="package://hexapod_description/meshes/leg_tibia.stl" mesh_scale="0.001 0.001 0.001" />
+						<m_joint_fixed name="leg2_tibia__leg2_rubber_tip" type="fixed"
+						 parent="leg2_tibia" child="leg2_rubber_tip" />
+						<m_rubber_tip_link name="leg2_rubber_tip"
+								origin_xyz="0 0.136283 -0.133814" origin_rpy="3.5185838 0 0"
+								inertia_origin_xyz="0.083874 0.000095 0.046294"
+								mesh_file="package://hexapod_description/meshes/leg_rubber_tip.stl" mesh_scale="0.001 0.001 0.001" />
 		<!-- LEG 3 (East) -->
 			<m_joint name="base_link__leg3_coxa" type="revolute" axis_xyz="0 0 1"
@@ -83,4 +95,10 @@
 							inertia_origin_xyz="0.083874 0.000095 0.046294"
 							mesh_file="package://hexapod_description/meshes/leg_tibia.stl" mesh_scale="0.001 0.001 0.001" />
+						<m_joint_fixed name="leg3_tibia__leg3_rubber_tip" type="fixed"
+						 parent="leg3_tibia" child="leg3_rubber_tip" />
+						<m_rubber_tip_link name="leg3_rubber_tip"
+								origin_xyz="0 0.136283 -0.133814" origin_rpy="3.5185838 0 0"
+								inertia_origin_xyz="0.083874 0.000095 0.046294"
+								mesh_file="package://hexapod_description/meshes/leg_rubber_tip.stl" mesh_scale="0.001 0.001 0.001" />
 		<!-- LEG 4 (West) -->
 			<m_joint name="base_link__leg4_coxa" type="revolute" axis_xyz="0 0 1"
@@ -107,4 +125,10 @@
 							inertia_origin_xyz="0.083874 0.000095 0.046294"
 							mesh_file="package://hexapod_description/meshes/leg_tibia.stl" mesh_scale="0.001 0.001 0.001" />
+						<m_joint_fixed name="leg4_tibia__leg4_rubber_tip" type="fixed"
+						 parent="leg4_tibia" child="leg4_rubber_tip" />
+						<m_rubber_tip_link name="leg4_rubber_tip"
+								origin_xyz="0 0.136283 -0.133814" origin_rpy="3.5185838 0 0"
+								inertia_origin_xyz="0.083874 0.000095 0.046294"
+								mesh_file="package://hexapod_description/meshes/leg_rubber_tip.stl" mesh_scale="0.001 0.001 0.001" />
 		<!-- LEG 5 (South East) -->
 			<m_joint name="base_link__leg5_coxa" type="revolute" axis_xyz="0 0 1"
@@ -131,4 +155,10 @@
 							inertia_origin_xyz="0.083874 0.000095 0.046294"
 							mesh_file="package://hexapod_description/meshes/leg_tibia.stl" mesh_scale="0.001 0.001 0.001" />
+						<m_joint_fixed name="leg5_tibia__leg5_rubber_tip" type="fixed"
+						 parent="leg5_tibia" child="leg5_rubber_tip" />
+						<m_rubber_tip_link name="leg5_rubber_tip"
+								origin_xyz="0 0.136283 -0.133814" origin_rpy="3.5185838 0 0"
+								inertia_origin_xyz="0.083874 0.000095 0.046294"
+								mesh_file="package://hexapod_description/meshes/leg_rubber_tip.stl" mesh_scale="0.001 0.001 0.001" />
 		<!-- LEG 6 (South West) -->
 			<m_joint name="base_link__leg6_coxa" type="revolute" axis_xyz="0 0 1"
@@ -155,3 +185,9 @@
 							inertia_origin_xyz="0.083874 0.000095 0.046294"
 							mesh_file="package://hexapod_description/meshes/leg_tibia.stl" mesh_scale="0.001 0.001 0.001" />
+						<m_joint_fixed name="leg6_tibia__leg6_rubber_tip" type="fixed"
+						 parent="leg6_tibia" child="leg6_rubber_tip" />
+						<m_rubber_tip_link name="leg6_rubber_tip"
+								origin_xyz="0 0.136283 -0.133814" origin_rpy="3.5185838 0 0"
+								inertia_origin_xyz="0.083874 0.000095 0.046294"
+								mesh_file="package://hexapod_description/meshes/leg_rubber_tip.stl" mesh_scale="0.001 0.001 0.001" />
 </robot>

File: hexapod_description/urdf/links_joints_macro.xacro (robot description, xacro)
@@ -101,4 +101,28 @@
 		</link>
 	</xacro:macro>
+	<xacro:macro name="m_rubber_tip_link" params="name origin_xyz origin_rpy inertia_origin_xyz mesh_file mesh_scale">
+		<link name="${name}">
+			<collision>
+				<origin xyz="${origin_xyz}" rpy="${origin_rpy}" />
+				<geometry>
+					<mesh filename="${mesh_file}" scale="${mesh_scale}" />
+				</geometry>
+			</collision>
+			<visual>
+				<origin xyz="${origin_xyz}" rpy="${origin_rpy}" />
+				<geometry>
+					<mesh filename="${mesh_file}" scale="${mesh_scale}" />
+				</geometry>
+				<material name="red" />
+			</visual>
+			<inertial>
+      			<origin xyz="${inertia_origin_xyz}" rpy="${origin_rpy}"/>
+      			<mass value="0.5"/>
+      			<inertia ixx="0.00126"	 	   ixy="0.000003599427"  ixz="-0.0007157"
+      					 iyx="0.000003599427"  iyy="0.001877" 		 iyz="0.000002060961"
+      					 izx="-0.0007157" 	   izy="0.000002060961"  izz="0.0008954"/>
+    		</inertial>
+		</link>
+	</xacro:macro>
 	<xacro:macro name="m_joint" params="name type axis_xyz effort lower upper velocity origin_xyz origin_rpy parent child damping" >
 		<joint name="${name}" type="${type}">
@@ -111,3 +135,9 @@
 		</joint>
 	</xacro:macro>
+	<xacro:macro name="m_joint_fixed" params="name type parent child" >
+		<joint name="${name}" type="${type}">
+			<parent link="${parent}" />
+			<child link="${child}" />
+		</joint>
+	</xacro:macro>
 </robot>
