Commit message: Added control

File: hexapod_description/urdf/hexapod_body.xacro (robot description, xacro)
@@ -3,191 +3,347 @@
 	<xacro:include filename="$(find hexapod_description)/urdf/links_joints_macro.xacro" />
 	<!-- Used for fixing robot to Gazebo 'base_link' -->
-		<link name="world"/>
- 		<joint name="fixed" type="fixed">
-  			<parent link="world"/>
+		<link name="base_dummy"/>
+ 		<joint name="fixed_joint" type="fixed">
+  			<parent link="base_dummy"/>
    			<child link="base_link"/>
- 		 </joint>
+   			<origin xyz="0 0 0" rpy="0 0 0"/>
+ 		</joint>
 		<m_base_link name="base_link"
-				origin_xyz="0 0 0" origin_rpy="0 0 0" inertia_origin_xyz="-0.00000000611 0.000002 0.021504"
-				mesh_file="package://hexapod_description/meshes/base_link.stl" mesh_scale="0.001 0.001 0.001" />
+				origin_xyz="0 0 0" origin_rpy="0 0 0" inertia_origin_xyz="0 0 0.021" />
 		<!-- LEG 1 (North East) -->
 			<m_joint name="base_link__leg1_coxa" type="revolute" axis_xyz="0 0 1"
-					 effort="1000.0" lower="-1.5708" upper="1.5708" velocity="0.5"
+					 effort="10000.0" lower="-1.5708" upper="1.5708" velocity="100"
 			 		 origin_xyz="0.072981 0.109608 0" origin_rpy="0 0 -0.7854"
 					 parent="base_link" child="leg1_coxa" damping="0.7"/>
 			<m_coxa_link name="leg1_coxa"
-					origin_xyz="0 0 0.021" origin_rpy="0 0 0" inertia_origin_xyz="0.00006 0.023937 0.00006"
-					mesh_file="package://hexapod_description/meshes/leg_coxa.stl" mesh_scale="0.001 0.001 0.001" />
+					origin_xyz="0 0 0.021" origin_rpy="0 0 0" inertia_origin_xyz="0 0.023937 0.021" />
 				<m_joint name="leg1_coxa__leg1_femur" type="revolute" axis_xyz="1 0 0"
-				 effort="1000.0" lower="-1.5708" upper="1.5708" velocity="0.5"
+				 effort="10000.0" lower="-1.5708" upper="1.5708" velocity="100"
 				 origin_xyz="0 0.047868 0.021" origin_rpy="0 0 0"
 				 parent="leg1_coxa" child="leg1_femur" damping="0.7"/>
 				<m_femur_link name="leg1_femur"
 						origin_xyz="0 0.0385 0" origin_rpy="0 3.14159 0"
-						inertia_origin_xyz="0.000216 -0.0000003648 -0.00000000863"
-						mesh_file="package://hexapod_description/meshes/leg_femur.stl" mesh_scale="0.001 0.001 0.001" />
+						inertia_origin_xyz="0 0.0385 0" />
 					<m_joint name="leg1_femur__leg1_tibia" type="revolute" axis_xyz="1 0 0"
-					 effort="1000.0" lower="-1.5708" upper="1.5708" velocity="0.5"
+					 effort="10000.0" lower="-1.5708" upper="1.5708" velocity="100"
 					 origin_xyz="0 0.077 0" origin_rpy="0 0 0"
 					 parent="leg1_femur" child="leg1_tibia" damping="0.7"/>
 					<m_tibia_link name="leg1_tibia"
 							origin_xyz="0 0 0" origin_rpy="3.14159 0 1.5708"
-							inertia_origin_xyz="0.083874 0.000095 0.046294"
-							mesh_file="package://hexapod_description/meshes/leg_tibia.stl" mesh_scale="0.001 0.001 0.001" />
+							inertia_origin_xyz="0 0.077796 -0.036156"/>
 						<m_joint_fixed name="leg1_tibia__leg1_rubber_tip" type="fixed"
 						 parent="leg1_tibia" child="leg1_rubber_tip" />
 						<m_rubber_tip_link name="leg1_rubber_tip"
 								origin_xyz="0 0.136283 -0.133814" origin_rpy="3.5185838 0 0"
-								inertia_origin_xyz="0.083874 0.000095 0.046294"
-								mesh_file="package://hexapod_description/meshes/leg_rubber_tip.stl" mesh_scale="0.001 0.001 0.001" />
+								inertia_origin_xyz="0 0.136283 -0.133814"/>
 		<!-- LEG 2 (North West) -->
 			<m_joint name="base_link__leg2_coxa" type="revolute" axis_xyz="0 0 1"
-					 effort="1000.0" lower="-1.5708" upper="1.5708" velocity="0.5"
+					 effort="10000.0" lower="-1.5708" upper="1.5708" velocity="100"
 			 		 origin_xyz="-0.072981 0.109608 0" origin_rpy="0 0 0.7854"
 					 parent="base_link" child="leg2_coxa" damping="0.7"/>
 			<m_coxa_link name="leg2_coxa"
-					origin_xyz="0 0 0.021" origin_rpy="0 0 0" inertia_origin_xyz="0.00006 0.023937 0.00006"
-					mesh_file="package://hexapod_description/meshes/leg_coxa.stl" mesh_scale="0.001 0.001 0.001" />
+					origin_xyz="0 0 0.021" origin_rpy="0 0 0" inertia_origin_xyz="0 0.023937 0.021"/>
 				<m_joint name="leg2_coxa__leg2_femur" type="revolute" axis_xyz="1 0 0"
-						 effort="1000.0" lower="-1.5708" upper="1.5708" velocity="0.5"
+						 effort="10000.0" lower="-1.5708" upper="1.5708" velocity="100"
 						 origin_xyz="0 0.047868 0.021" origin_rpy="0 0 0"
 						 parent="leg2_coxa" child="leg2_femur" damping="0.7"/>
 				<m_femur_link name="leg2_femur"
 						origin_xyz="0 0.0385 0" origin_rpy="0 3.14159 0"
-						inertia_origin_xyz="0.000216 -0.0000003648 -0.00000000863"
-						mesh_file="package://hexapod_description/meshes/leg_femur.stl" mesh_scale="0.001 0.001 0.001" />
+						inertia_origin_xyz="0 0.0385 0"/>
 					<m_joint name="leg2_femur__leg2_tibia" type="revolute" axis_xyz="1 0 0"
-					 effort="1000.0" lower="-1.5708" upper="1.5708" velocity="0.5"
+					 effort="10000.0" lower="-1.5708" upper="1.5708" velocity="100"
 					 origin_xyz="0 0.077 0" origin_rpy="0 0 0"
 					 parent="leg2_femur" child="leg2_tibia" damping="0.7"/>
 					<m_tibia_link name="leg2_tibia"
 							origin_xyz="0 0 0" origin_rpy="3.14159 0 1.5708"
-							inertia_origin_xyz="0.083874 0.000095 0.046294"
-							mesh_file="package://hexapod_description/meshes/leg_tibia.stl" mesh_scale="0.001 0.001 0.001" />
+							inertia_origin_xyz="0 0.077796 -0.036156"/>
 						<m_joint_fixed name="leg2_tibia__leg2_rubber_tip" type="fixed"
 						 parent="leg2_tibia" child="leg2_rubber_tip" />
 						<m_rubber_tip_link name="leg2_rubber_tip"
 								origin_xyz="0 0.136283 -0.133814" origin_rpy="3.5185838 0 0"
-								inertia_origin_xyz="0.083874 0.000095 0.046294"
-								mesh_file="package://hexapod_description/meshes/leg_rubber_tip.stl" mesh_scale="0.001 0.001 0.001" />
+								inertia_origin_xyz="0 0.136283 -0.133814"/>
 		<!-- LEG 3 (East) -->
 			<m_joint name="base_link__leg3_coxa" type="revolute" axis_xyz="0 0 1"
-					 effort="1000.0" lower="-1.5708" upper="1.5708" velocity="0.5"
+					 effort="10000.0" lower="-1.5708" upper="1.5708" velocity="100"
 			 		 origin_xyz="0.09850 0 0" origin_rpy="0 0 -1.5708"
 					 parent="base_link" child="leg3_coxa" damping="0.7"/>
-			<m_coxa_link name="leg3_coxa" inertia_origin_xyz="0.00006 0.023937 0.00006"
-					origin_xyz="0 0 0.021" origin_rpy="0 0 0"
-					mesh_file="package://hexapod_description/meshes/leg_coxa.stl" mesh_scale="0.001 0.001 0.001" />
+			<m_coxa_link name="leg3_coxa" inertia_origin_xyz="0 0.023937 0.021"
+					origin_xyz="0 0 0.021" origin_rpy="0 0 0"/>
 				<m_joint name="leg3_coxa__leg3_femur" type="revolute" axis_xyz="1 0 0"
-						 effort="1000.0" lower="-1.5708" upper="1.5708" velocity="0.5"
+						 effort="10000.0" lower="-1.5708" upper="1.5708" velocity="100"
 						 origin_xyz="0 0.047868 0.021" origin_rpy="0 0 0"
 						 parent="leg3_coxa" child="leg3_femur" damping="0.7"/>
 				<m_femur_link name="leg3_femur"
 						origin_xyz="0 0.0385 0" origin_rpy="0 3.14159 0"
-						inertia_origin_xyz="0.000216 -0.0000003648 -0.00000000863"
-						mesh_file="package://hexapod_description/meshes/leg_femur.stl" mesh_scale="0.001 0.001 0.001" />
+						inertia_origin_xyz="0 0.0385 0"/>
 					<m_joint name="leg3_femur__leg3_tibia" type="revolute" axis_xyz="1 0 0"
-					 effort="1000.0" lower="-1.5708" upper="1.5708" velocity="0.5"
+					 effort="10000.0" lower="-1.5708" upper="1.5708" velocity="100"
 					 origin_xyz="0 0.077 0" origin_rpy="0 0 0"
 					 parent="leg3_femur" child="leg3_tibia" damping="0.7"/>
 					<m_tibia_link name="leg3_tibia"
 							origin_xyz="0 0 0" origin_rpy="3.14159 0 1.5708"
-							inertia_origin_xyz="0.083874 0.000095 0.046294"
-							mesh_file="package://hexapod_description/meshes/leg_tibia.stl" mesh_scale="0.001 0.001 0.001" />
+							inertia_origin_xyz="0 0.077796 -0.036156"/>
 						<m_joint_fixed name="leg3_tibia__leg3_rubber_tip" type="fixed"
 						 parent="leg3_tibia" child="leg3_rubber_tip" />
 						<m_rubber_tip_link name="leg3_rubber_tip"
 								origin_xyz="0 0.136283 -0.133814" origin_rpy="3.5185838 0 0"
-								inertia_origin_xyz="0.083874 0.000095 0.046294"
-								mesh_file="package://hexapod_description/meshes/leg_rubber_tip.stl" mesh_scale="0.001 0.001 0.001" />
+								inertia_origin_xyz="0 0.136283 -0.133814"/>
 		<!-- LEG 4 (West) -->
 			<m_joint name="base_link__leg4_coxa" type="revolute" axis_xyz="0 0 1"
-					 effort="1000.0" lower="-1.5708" upper="1.5708" velocity="0.5"
+					 effort="10000.0" lower="-1.5708" upper="1.5708" velocity="100"
 			 		 origin_xyz="-0.09850 0 0" origin_rpy="0 0 1.5708"
 					 parent="base_link" child="leg4_coxa" damping="0.7"/>
 			<m_coxa_link name="leg4_coxa"
-					origin_xyz="0 0 0.021" origin_rpy="0 0 0" inertia_origin_xyz="0.00006 0.023937 0.00006"
-					mesh_file="package://hexapod_description/meshes/leg_coxa.stl" mesh_scale="0.001 0.001 0.001" />
+					origin_xyz="0 0 0.021" origin_rpy="0 0 0" inertia_origin_xyz="0 0.023937 0.021"/>
 				<m_joint name="leg4_coxa__leg4_femur" type="revolute" axis_xyz="1 0 0"
-				 effort="1000.0" lower="-1.5708" upper="1.5708" velocity="0.5"
+				 effort="10000.0" lower="-1.5708" upper="1.5708" velocity="100"
 				 origin_xyz="0 0.047868 0.021" origin_rpy="0 0 0"
 				 parent="leg4_coxa" child="leg4_femur" damping="0.7"/>
 				<m_femur_link name="leg4_femur"
 						origin_xyz="0 0.0385 0" origin_rpy="0 3.14159 0"
-						inertia_origin_xyz="0.000216 -0.0000003648 -0.00000000863"
-						mesh_file="package://hexapod_description/meshes/leg_femur.stl" mesh_scale="0.001 0.001 0.001" />
+						inertia_origin_xyz="0 0.0385 0"/>
 					<m_joint name="leg4_femur__leg4_tibia" type="revolute" axis_xyz="1 0 0"
-					 effort="1000.0" lower="-1.5708" upper="1.5708" velocity="0.5"
+					 effort="10000.0" lower="-1.5708" upper="1.5708" velocity="100"
 					 origin_xyz="0 0.077 0" origin_rpy="0 0 0"
 					 parent="leg4_femur" child="leg4_tibia" damping="0.7"/>
 					<m_tibia_link name="leg4_tibia"
 							origin_xyz="0 0 0" origin_rpy="3.14159 0 1.5708"
-							inertia_origin_xyz="0.083874 0.000095 0.046294"
-							mesh_file="package://hexapod_description/meshes/leg_tibia.stl" mesh_scale="0.001 0.001 0.001" />
+							inertia_origin_xyz="0 0.077796 -0.036156"/>
 						<m_joint_fixed name="leg4_tibia__leg4_rubber_tip" type="fixed"
 						 parent="leg4_tibia" child="leg4_rubber_tip" />
 						<m_rubber_tip_link name="leg4_rubber_tip"
 								origin_xyz="0 0.136283 -0.133814" origin_rpy="3.5185838 0 0"
-								inertia_origin_xyz="0.083874 0.000095 0.046294"
-								mesh_file="package://hexapod_description/meshes/leg_rubber_tip.stl" mesh_scale="0.001 0.001 0.001" />
+								inertia_origin_xyz="0 0.136283 -0.133814"/>
 		<!-- LEG 5 (South East) -->
 			<m_joint name="base_link__leg5_coxa" type="revolute" axis_xyz="0 0 1"
-					 effort="1000.0" lower="-1.5708" upper="1.5708" velocity="0.5"
+					 effort="10000.0" lower="-1.5708" upper="1.5708" velocity="100"
 			 		 origin_xyz="0.072981 -0.109608 0" origin_rpy="0 0 -2.3562"
 					 parent="base_link" child="leg5_coxa" damping="0.7"/>
 			<m_coxa_link name="leg5_coxa"
-					origin_xyz="0 0 0.021" origin_rpy="0 0 0" inertia_origin_xyz="0.00006 0.023937 0.00006"
-					mesh_file="package://hexapod_description/meshes/leg_coxa.stl" mesh_scale="0.001 0.001 0.001" />
+					origin_xyz="0 0 0.021" origin_rpy="0 0 0" inertia_origin_xyz="0 0.023937 0.021"/>
 				<m_joint name="leg5_coxa__leg5_femur" type="revolute" axis_xyz="1 0 0"
-						 effort="1000.0" lower="-1.5708" upper="1.5708" velocity="0.5"
+						 effort="10000.0" lower="-1.5708" upper="1.5708" velocity="100"
 						 origin_xyz="0 0.047868 0.021" origin_rpy="0 0 0"
 						 parent="leg5_coxa" child="leg5_femur" damping="0.7"/>
 				<m_femur_link name="leg5_femur"
 						origin_xyz="0 0.0385 0" origin_rpy="0 3.14159 0"
-						inertia_origin_xyz="0.000216 -0.0000003648 -0.00000000863"
-						mesh_file="package://hexapod_description/meshes/leg_femur.stl" mesh_scale="0.001 0.001 0.001" />
+						inertia_origin_xyz="0 0.0385 0"/>
 					<m_joint name="leg5_femur__leg5_tibia" type="revolute" axis_xyz="1 0 0"
-					 effort="1000.0" lower="-1.5708" upper="1.5708" velocity="0.5"
+					 effort="10000.0" lower="-1.5708" upper="1.5708" velocity="100"
 					 origin_xyz="0 0.077 0" origin_rpy="0 0 0"
 					 parent="leg5_femur" child="leg5_tibia" damping="0.7"/>
 					<m_tibia_link name="leg5_tibia"
 							origin_xyz="0 0 0" origin_rpy="3.14159 0 1.5708"
-							inertia_origin_xyz="0.083874 0.000095 0.046294"
-							mesh_file="package://hexapod_description/meshes/leg_tibia.stl" mesh_scale="0.001 0.001 0.001" />
+							inertia_origin_xyz="0 0.077796 -0.036156"/>
 						<m_joint_fixed name="leg5_tibia__leg5_rubber_tip" type="fixed"
 						 parent="leg5_tibia" child="leg5_rubber_tip" />
 						<m_rubber_tip_link name="leg5_rubber_tip"
 								origin_xyz="0 0.136283 -0.133814" origin_rpy="3.5185838 0 0"
-								inertia_origin_xyz="0.083874 0.000095 0.046294"
-								mesh_file="package://hexapod_description/meshes/leg_rubber_tip.stl" mesh_scale="0.001 0.001 0.001" />
+								inertia_origin_xyz="0 0.136283 -0.133814"/>
 		<!-- LEG 6 (South West) -->
 			<m_joint name="base_link__leg6_coxa" type="revolute" axis_xyz="0 0 1"
-					 effort="1000.0" lower="-1.5708" upper="1.5708" velocity="0.5"
+					 effort="10000.0" lower="-1.5708" upper="1.5708" velocity="100"
 			 		 origin_xyz="-0.072981 -0.109608 0" origin_rpy="0 0 2.3562"
 					 parent="base_link" child="leg6_coxa" damping="0.7"/>
 			<m_coxa_link name="leg6_coxa"
-					origin_xyz="0 0 0.021" origin_rpy="0 0 0" inertia_origin_xyz="0.00006 0.023937 0.00006"
-					mesh_file="package://hexapod_description/meshes/leg_coxa.stl" mesh_scale="0.001 0.001 0.001" />
+					origin_xyz="0 0 0.021" origin_rpy="0 0 0" inertia_origin_xyz="0 0.023937 0.021"/>
 				<m_joint name="leg6_coxa__leg6_femur" type="revolute" axis_xyz="1 0 0"
-						 effort="1000.0" lower="-1.5708" upper="1.5708" velocity="0.5"
+						 effort="10000.0" lower="-1.5708" upper="1.5708" velocity="100"
 						 origin_xyz="0 0.047868 0.021" origin_rpy="0 0 0"
 						 parent="leg6_coxa" child="leg6_femur" damping="0.7"/>
 				<m_femur_link name="leg6_femur"
 						origin_xyz="0 0.0385 0" origin_rpy="0 3.14159 0"
-						inertia_origin_xyz="0.000216 -0.0000003648 -0.00000000863"
-						mesh_file="package://hexapod_description/meshes/leg_femur.stl" mesh_scale="0.001 0.001 0.001" />
+						inertia_origin_xyz="0 0.0385 0"/>
 					<m_joint name="leg6_femur__leg6_tibia" type="revolute" axis_xyz="1 0 0"
-					 effort="1000.0" lower="-1.5708" upper="1.5708" velocity="0.5"
+					 effort="10000.0" lower="-1.5708" upper="1.5708" velocity="100"
 					 origin_xyz="0 0.077 0" origin_rpy="0 0 0"
 					 parent="leg6_femur" child="leg6_tibia" damping="0.7"/>
 					<m_tibia_link name="leg6_tibia"
 							origin_xyz="0 0 0" origin_rpy="3.14159 0 1.5708"
-							inertia_origin_xyz="0.083874 0.000095 0.046294"
-							mesh_file="package://hexapod_description/meshes/leg_tibia.stl" mesh_scale="0.001 0.001 0.001" />
+							inertia_origin_xyz="0 0.077796 -0.036156"/>
 						<m_joint_fixed name="leg6_tibia__leg6_rubber_tip" type="fixed"
 						 parent="leg6_tibia" child="leg6_rubber_tip" />
 						<m_rubber_tip_link name="leg6_rubber_tip"
 								origin_xyz="0 0.136283 -0.133814" origin_rpy="3.5185838 0 0"
-								inertia_origin_xyz="0.083874 0.000095 0.046294"
-								mesh_file="package://hexapod_description/meshes/leg_rubber_tip.stl" mesh_scale="0.001 0.001 0.001" />
+								inertia_origin_xyz="0 0.136283 -0.133814"/>
+	<transmission name ="trans_base_link__leg1_coxa">
+		<type>transmission_interface/SimpleTransmission</type>
+		<joint name="base_link__leg1_coxa">
+			<hardwareInterface>EffortJointInterface</hardwareInterface>
+		</joint>
+		<actuator name="motor_base_link__leg1_coxa">
+			<hardwareInterface>EffortJointInterface</hardwareInterface>
+			<mechanicalReduction>1</mechanicalReduction>
+		</actuator>
+	</transmission>
+	<transmission name ="trans_leg1_coxa__leg1_femur">
+		<type>transmission_interface/SimpleTransmission</type>
+		<joint name="leg1_coxa__leg1_femur">
+			<hardwareInterface>EffortJointInterface</hardwareInterface>
+		</joint>
+		<actuator name="motor_leg1_coxa__leg1_femur">
+			<hardwareInterface>EffortJointInterface</hardwareInterface>
+			<mechanicalReduction>1</mechanicalReduction>
+		</actuator>
+	</transmission>
+	<transmission name ="trans_leg1_femur__leg1_tibia">
+		<type>transmission_interface/SimpleTransmission</type>
+		<joint name="leg1_femur__leg1_tibia">
+			<hardwareInterface>EffortJointInterface</hardwareInterface>
+		</joint>
+		<actuator name="motor_leg1_femur__leg1_tibia">
+			<hardwareInterface>EffortJointInterface</hardwareInterface>
+			<mechanicalReduction>1</mechanicalReduction>
+		</actuator>
+	</transmission>
+	<transmission name ="trans_base_link__leg2_coxa">
+		<type>transmission_interface/SimpleTransmission</type>
+		<joint name="base_link__leg2_coxa">
+			<hardwareInterface>EffortJointInterface</hardwareInterface>
+		</joint>
+		<actuator name="motor_base_link__leg2_coxa">
+			<hardwareInterface>EffortJointInterface</hardwareInterface>
+			<mechanicalReduction>1</mechanicalReduction>
+		</actuator>
+	</transmission>
+	<transmission name ="trans_leg2_coxa__leg2_femur">
+		<type>transmission_interface/SimpleTransmission</type>
+		<joint name="leg2_coxa__leg2_femur">
+			<hardwareInterface>EffortJointInterface</hardwareInterface>
+		</joint>
+		<actuator name="motor_leg2_coxa__leg2_femur">
+			<hardwareInterface>EffortJointInterface</hardwareInterface>
+			<mechanicalReduction>1</mechanicalReduction>
+		</actuator>
+	</transmission>
+	<transmission name ="trans_leg2_femur__leg2_tibia">
+		<type>transmission_interface/SimpleTransmission</type>
+		<joint name="leg2_femur__leg2_tibia">
+			<hardwareInterface>EffortJointInterface</hardwareInterface>
+		</joint>
+		<actuator name="motor_leg2_femur__leg2_tibia">
+			<hardwareInterface>EffortJointInterface</hardwareInterface>
+			<mechanicalReduction>1</mechanicalReduction>
+		</actuator>
+	</transmission>
+	<transmission name ="trans_base_link__leg3_coxa">
+		<type>transmission_interface/SimpleTransmission</type>
+		<joint name="base_link__leg3_coxa">
+			<hardwareInterface>EffortJointInterface</hardwareInterface>
+		</joint>
+		<actuator name="motor_base_link__leg3_coxa">
+			<hardwareInterface>EffortJointInterface</hardwareInterface>
+			<mechanicalReduction>1</mechanicalReduction>
+		</actuator>
+	</transmission>
+	<transmission name ="trans_leg3_coxa__leg3_femur">
+		<type>transmission_interface/SimpleTransmission</type>
+		<joint name="leg3_coxa__leg3_femur">
+			<hardwareInterface>EffortJointInterface</hardwareInterface>
+		</joint>
+		<actuator name="motor_leg3_coxa__leg3_femur">
+			<hardwareInterface>EffortJointInterface</hardwareInterface>
+			<mechanicalReduction>1</mechanicalReduction>
+		</actuator>
+	</transmission>
+	<transmission name ="trans_leg3_femur__leg3_tibia">
+		<type>transmission_interface/SimpleTransmission</type>
+		<joint name="leg3_femur__leg3_tibia">
+			<hardwareInterface>EffortJointInterface</hardwareInterface>
+		</joint>
+		<actuator name="motor_leg3_femur__leg3_tibia">
+			<hardwareInterface>EffortJointInterface</hardwareInterface>
+			<mechanicalReduction>1</mechanicalReduction>
+		</actuator>
+	</transmission>
+	<transmission name ="trans_base_link__leg4_coxa">
+		<type>transmission_interface/SimpleTransmission</type>
+		<joint name="base_link__leg4_coxa">
+			<hardwareInterface>EffortJointInterface</hardwareInterface>
+		</joint>
+		<actuator name="motor_base_link__leg4_coxa">
+			<hardwareInterface>EffortJointInterface</hardwareInterface>
+			<mechanicalReduction>1</mechanicalReduction>
+		</actuator>
+	</transmission>
+	<transmission name ="trans_leg4_coxa__leg4_femur">
+		<type>transmission_interface/SimpleTransmission</type>
+		<joint name="leg4_coxa__leg4_femur">
+			<hardwareInterface>EffortJointInterface</hardwareInterface>
+		</joint>
+		<actuator name="motor_leg4_coxa__leg4_femur">
+			<hardwareInterface>EffortJointInterface</hardwareInterface>
+			<mechanicalReduction>1</mechanicalReduction>
+		</actuator>
+	</transmission>
+	<transmission name ="trans_leg4_femur__leg4_tibia">
+		<type>transmission_interface/SimpleTransmission</type>
+		<joint name="leg4_femur__leg4_tibia">
+			<hardwareInterface>EffortJointInterface</hardwareInterface>
+		</joint>
+		<actuator name="motor_leg4_femur__leg4_tibia">
+			<hardwareInterface>EffortJointInterface</hardwareInterface>
+			<mechanicalReduction>1</mechanicalReduction>
+		</actuator>
+	</transmission>
+	<transmission name ="trans_base_link__leg5_coxa">
+		<type>transmission_interface/SimpleTransmission</type>
+		<joint name="base_link__leg5_coxa">
+			<hardwareInterface>EffortJointInterface</hardwareInterface>
+		</joint>
+		<actuator name="motor_base_link__leg5_coxa">
+			<hardwareInterface>EffortJointInterface</hardwareInterface>
+			<mechanicalReduction>1</mechanicalReduction>
+		</actuator>
+	</transmission>
+	<transmission name ="trans_leg5_coxa__leg5_femur">
+		<type>transmission_interface/SimpleTransmission</type>
+		<joint name="leg5_coxa__leg5_femur">
+			<hardwareInterface>EffortJointInterface</hardwareInterface>
+		</joint>
+		<actuator name="motor_leg5_coxa__leg5_femur">
+			<hardwareInterface>EffortJointInterface</hardwareInterface>
+			<mechanicalReduction>1</mechanicalReduction>
+		</actuator>
+	</transmission>
+	<transmission name ="trans_leg5_femur__leg5_tibia">
+		<type>transmission_interface/SimpleTransmission</type>
+		<joint name="leg5_femur__leg5_tibia">
+			<hardwareInterface>EffortJointInterface</hardwareInterface>
+		</joint>
+		<actuator name="motor_leg5_femur__leg5_tibia">
+			<hardwareInterface>EffortJointInterface</hardwareInterface>
+			<mechanicalReduction>1</mechanicalReduction>
+		</actuator>
+	</transmission>
+	<transmission name ="trans_base_link__leg6_coxa">
+		<type>transmission_interface/SimpleTransmission</type>
+		<joint name="base_link__leg6_coxa">
+			<hardwareInterface>EffortJointInterface</hardwareInterface>
+		</joint>
+		<actuator name="motor_base_link__leg6_coxa">
+			<hardwareInterface>EffortJointInterface</hardwareInterface>
+			<mechanicalReduction>1</mechanicalReduction>
+		</actuator>
+	</transmission>
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