Commit message: Added control

File: hexapod_description/urdf/links_joints_macro.xacro (robot description, xacro)
@@ -5,10 +5,10 @@
   <!-- Import Rviz colors -->
   <xacro:include filename="$(find hexapod_description)/urdf/materials.xacro" />
-	<xacro:macro name="m_base_link" params="name origin_xyz origin_rpy inertia_origin_xyz mesh_file mesh_scale">
+	<xacro:macro name="m_base_link" params="name origin_xyz origin_rpy inertia_origin_xyz">
 		<link name="${name}">
 			<collision>
 				<origin xyz="${origin_xyz}" rpy="${origin_rpy}" />
 				<geometry>
-					<mesh filename="${mesh_file}" scale="${mesh_scale}" />
+					<mesh filename="package://hexapod_description/meshes/base_link_collision.stl" scale="0.001 0.001 0.001" />
 				</geometry>
 			</collision>
@@ -16,5 +16,29 @@
 				<origin xyz="${origin_xyz}" rpy="${origin_rpy}" />
 				<geometry>
-					<mesh filename="${mesh_file}" scale="${mesh_scale}" />
+					<mesh filename="package://hexapod_description/meshes/base_link.stl" scale="0.001 0.001 0.001" />
+				</geometry>
+				<material name="red" />
+			</visual>
+			<inertial>
+      			<origin xyz="${inertia_origin_xyz}" rpy="0 0 0"/>
+      			<mass value="1.3"/>
+      			<inertia ixx="5.404e-3"			ixy="0" 			ixz="0"
+      					 iyx="0"				iyy="3.169e-3" 		iyz="0"
+      					 izx="0"  				izy="0" 			izz="8.191e-3"/>
+    		</inertial>
+		</link>
+	</xacro:macro>
+	<xacro:macro name="m_coxa_link" params="name origin_xyz origin_rpy inertia_origin_xyz">
+		<link name="${name}">
+			<collision>
+				<origin xyz="${origin_xyz}" rpy="${origin_rpy}" />
+				<geometry>
+					<mesh filename="package://hexapod_description/meshes/leg_coxa_collision.stl" scale="0.001 0.001 0.001" />
+				</geometry>
+			</collision>
+			<visual>
+				<origin xyz="${origin_xyz}" rpy="${origin_rpy}" />
+				<geometry>
+					<mesh filename="package://hexapod_description/meshes/leg_coxa.stl" scale="0.001 0.001 0.001" />
 				</geometry>
 				<material name="red" />
@@ -22,17 +46,17 @@
 			<inertial>
       			<origin xyz="${inertia_origin_xyz}" rpy="${origin_rpy}"/>
-      			<mass value="4"/>
-      			<inertia ixx="0.02109" 		   ixy="-0.000000524323" ixz="0.000000000016"
-      					 iyx="-0.000000524323" iyy="0.0144" 		 iyz="0.000003891"
-      					 izx="0.000000000016"  izy="0.000003891" 	 izz="0.0373"/>
+      			<mass value="0.04"/>
+      			<inertia ixx="1.605e-5"			ixy="-5.7988e-8"		ixz="0"
+      					 iyx="-5.7988e-8"		iyy="2.012e-5"			iyz="5.7639e-8"
+      					 izx="0"				izy="5.7639e-8"			izz="1.605e-5"/>
     		</inertial>
 		</link>
 	</xacro:macro>
-	<xacro:macro name="m_coxa_link" params="name origin_xyz origin_rpy inertia_origin_xyz mesh_file mesh_scale">
+	<xacro:macro name="m_femur_link" params="name origin_xyz origin_rpy inertia_origin_xyz">
 		<link name="${name}">
 			<collision>
 				<origin xyz="${origin_xyz}" rpy="${origin_rpy}" />
 				<geometry>
-					<mesh filename="${mesh_file}" scale="${mesh_scale}" />
+					<mesh filename="package://hexapod_description/meshes/leg_femur_collision.stl" scale="0.001 0.001 0.001" />
 				</geometry>
 			</collision>
@@ -40,5 +64,29 @@
 				<origin xyz="${origin_xyz}" rpy="${origin_rpy}" />
 				<geometry>
-					<mesh filename="${mesh_file}" scale="${mesh_scale}" />
+					<mesh filename="package://hexapod_description/meshes/leg_femur.stl" scale="0.001 0.001 0.001" />
+				</geometry>
+				<material name="red" />
+			</visual>
+			<inertial>
+      			<origin xyz="${inertia_origin_xyz}" rpy="0 0 0"/>
+      			<mass value="0.12"/>
+      			<inertia ixx="1.005e-4"			ixy="0"				ixz="0"
+      					 iyx="0"  				iyy="2.532e-5"		iyz="0"
+      					 izx="0"				izy="0"				izz="1.071e-4"/>
+    		</inertial>
+		</link>
+	</xacro:macro>
+	<xacro:macro name="m_tibia_link" params="name origin_xyz origin_rpy inertia_origin_xyz">
+		<link name="${name}">
+			<collision>
+				<origin xyz="${origin_xyz}" rpy="${origin_rpy}" />
+				<geometry>
+					<mesh filename="package://hexapod_description/meshes/leg_tibia_collision.stl" scale="0.001 0.001 0.001" />
+				</geometry>
+			</collision>
+			<visual>
+				<origin xyz="${origin_xyz}" rpy="${origin_rpy}" />
+				<geometry>
+					<mesh filename="package://hexapod_description/meshes/leg_tibia.stl" scale="0.001 0.001 0.001" />
 				</geometry>
 				<material name="red" />
@@ -46,17 +94,17 @@
 			<inertial>
       			<origin xyz="${inertia_origin_xyz}" rpy="${origin_rpy}"/>
-      			<mass value="0.2"/>
-      			<inertia ixx="0.00008176" 	   ixy="-0.000000295397" ixz="0.000000000742"
-      					 iyx="-0.000000295397" iyy="0.0001025" 		 iyz="0.000000293619"
-      					 izx="0.000000000742"  izy="0.000000293619"  izz="0.00008176"/>
+      			<mass value="0.098"/>
+      			<inertia ixx="1.515e-4"			ixy="1.52255e-7"			ixz="-9.144e-5"
+      					 iyx="1.52255e-7"  		iyy="2.328e-4"				iyz="7.0753e-8"
+      					 izx="-9.144e-5"		izy="7.0753e-8"				izz="1.159e-4"/>
     		</inertial>
 		</link>
 	</xacro:macro>
-	<xacro:macro name="m_femur_link" params="name origin_xyz origin_rpy inertia_origin_xyz mesh_file mesh_scale">
+	<xacro:macro name="m_rubber_tip_link" params="name origin_xyz origin_rpy inertia_origin_xyz">
 		<link name="${name}">
 			<collision>
 				<origin xyz="${origin_xyz}" rpy="${origin_rpy}" />
 				<geometry>
-					<mesh filename="${mesh_file}" scale="${mesh_scale}" />
+					<mesh filename="package://hexapod_description/meshes/leg_rubber_tip.stl" scale="0.001 0.001 0.001" />
 				</geometry>
 			</collision>
@@ -64,5 +112,5 @@
 				<origin xyz="${origin_xyz}" rpy="${origin_rpy}" />
 				<geometry>
-					<mesh filename="${mesh_file}" scale="${mesh_scale}" />
+					<mesh filename="package://hexapod_description/meshes/leg_rubber_tip.stl" scale="0.001 0.001 0.001" />
 				</geometry>
 				<material name="red" />
@@ -70,56 +118,8 @@
 			<inertial>
       			<origin xyz="${inertia_origin_xyz}" rpy="${origin_rpy}"/>
-      			<mass value="0.7"/>
-      			<inertia ixx="0.0000616" 	   ixy="0.000000004936"  ixz="-0.000000000097"
-      					 iyx="0.000000004936"  iyy="0.0001212" 		 iyz="0.000000357772"
-      					 izx="-0.000000000097" izy="0.000000357772"  izz="0.0006537"/>
-    		</inertial>
-		</link>
-	</xacro:macro>
-	<xacro:macro name="m_tibia_link" params="name origin_xyz origin_rpy inertia_origin_xyz mesh_file mesh_scale">
-		<link name="${name}">
-			<collision>
-				<origin xyz="${origin_xyz}" rpy="${origin_rpy}" />
-				<geometry>
-					<mesh filename="${mesh_file}" scale="${mesh_scale}" />
-				</geometry>
-			</collision>
-			<visual>
-				<origin xyz="${origin_xyz}" rpy="${origin_rpy}" />
-				<geometry>
-					<mesh filename="${mesh_file}" scale="${mesh_scale}" />
-				</geometry>
-				<material name="red" />
-			</visual>
-			<inertial>
-      			<origin xyz="${inertia_origin_xyz}" rpy="${origin_rpy}"/>
-      			<mass value="0.5"/>
-      			<inertia ixx="0.00126"	 	   ixy="0.000003599427"  ixz="-0.0007157"
-      					 iyx="0.000003599427"  iyy="0.001877" 		 iyz="0.000002060961"
-      					 izx="-0.0007157" 	   izy="0.000002060961"  izz="0.0008954"/>
-    		</inertial>
-		</link>
-	</xacro:macro>
-	<xacro:macro name="m_rubber_tip_link" params="name origin_xyz origin_rpy inertia_origin_xyz mesh_file mesh_scale">
-		<link name="${name}">
-			<collision>
-				<origin xyz="${origin_xyz}" rpy="${origin_rpy}" />
-				<geometry>
-					<mesh filename="${mesh_file}" scale="${mesh_scale}" />
-				</geometry>
-			</collision>
-			<visual>
-				<origin xyz="${origin_xyz}" rpy="${origin_rpy}" />
-				<geometry>
-					<mesh filename="${mesh_file}" scale="${mesh_scale}" />
-				</geometry>
-				<material name="red" />
-			</visual>
-			<inertial>
-      			<origin xyz="${inertia_origin_xyz}" rpy="${origin_rpy}"/>
-      			<mass value="0.5"/>
-      			<inertia ixx="0.00126"	 	   ixy="0.000003599427"  ixz="-0.0007157"
-      					 iyx="0.000003599427"  iyy="0.001877" 		 iyz="0.000002060961"
-      					 izx="-0.0007157" 	   izy="0.000002060961"  izz="0.0008954"/>
+      			<mass value="0.002"/>
+      			<inertia ixx="1.00584e-7" 			ixy="0" 			ixz="0"
+      					 iyx="0"  					iyy="1.00579e-7"	iyz="0"
+      					 izx="0" 					izy="0" 			izz="1.05103e-7"/>
     		</inertial>
 		</link>

Commit message: Added teleop_joy

File: hexapod_description/urdf/hexapod_body.xacro (robot description, xacro)
@@ -13,20 +13,20 @@
 		<!-- LEG 1 (North East) -->
 			<m_joint name="base_link__leg1_coxa" type="revolute" axis_xyz="0 0 1"
-					 effort="10000.0" lower="-1.5708" upper="1.5708" velocity="100"
+					 effort="2.8" lower="-1.5708" upper="1.5708" velocity="5.6548668"
 			 		 origin_xyz="0.072981 0.109608 0" origin_rpy="0 0 -0.7854"
-					 parent="base_link" child="leg1_coxa" damping="0.7"/>
+					 parent="base_link" child="leg1_coxa" />
 			<m_coxa_link name="leg1_coxa"
 					origin_xyz="0 0 0.021" origin_rpy="0 0 0" inertia_origin_xyz="0 0.023937 0.021" />
 				<m_joint name="leg1_coxa__leg1_femur" type="revolute" axis_xyz="1 0 0"
-				 effort="10000.0" lower="-1.5708" upper="1.5708" velocity="100"
+				 effort="2.8" lower="-1.5708" upper="1.5708" velocity="5.6548668"
 				 origin_xyz="0 0.047868 0.021" origin_rpy="0 0 0"
-				 parent="leg1_coxa" child="leg1_femur" damping="0.7"/>
+				 parent="leg1_coxa" child="leg1_femur" />
 				<m_femur_link name="leg1_femur"
 						origin_xyz="0 0.0385 0" origin_rpy="0 3.14159 0"
 						inertia_origin_xyz="0 0.0385 0" />
 					<m_joint name="leg1_femur__leg1_tibia" type="revolute" axis_xyz="1 0 0"
-					 effort="10000.0" lower="-1.5708" upper="1.5708" velocity="100"
-					 origin_xyz="0 0.077 0" origin_rpy="0 0 0"
-					 parent="leg1_femur" child="leg1_tibia" damping="0.7"/>
+					 effort="2.8" lower="-1.5708" upper="1.5708" velocity="5.6548668"
+					 origin_xyz="0 0.077 0" origin_rpy="0 0 0"
+					 parent="leg1_femur" child="leg1_tibia" />
 					<m_tibia_link name="leg1_tibia"
 							origin_xyz="0 0 0" origin_rpy="3.14159 0 1.5708"
@@ -39,20 +39,20 @@
 		<!-- LEG 2 (North West) -->
 			<m_joint name="base_link__leg2_coxa" type="revolute" axis_xyz="0 0 1"
-					 effort="10000.0" lower="-1.5708" upper="1.5708" velocity="100"
+					 effort="2.8" lower="-1.5708" upper="1.5708" velocity="5.6548668"
 			 		 origin_xyz="-0.072981 0.109608 0" origin_rpy="0 0 0.7854"
-					 parent="base_link" child="leg2_coxa" damping="0.7"/>
+					 parent="base_link" child="leg2_coxa" />
 			<m_coxa_link name="leg2_coxa"
 					origin_xyz="0 0 0.021" origin_rpy="0 0 0" inertia_origin_xyz="0 0.023937 0.021"/>
 				<m_joint name="leg2_coxa__leg2_femur" type="revolute" axis_xyz="1 0 0"
-						 effort="10000.0" lower="-1.5708" upper="1.5708" velocity="100"
+						 effort="2.8" lower="-1.5708" upper="1.5708" velocity="5.6548668"
 						 origin_xyz="0 0.047868 0.021" origin_rpy="0 0 0"
-						 parent="leg2_coxa" child="leg2_femur" damping="0.7"/>
+						 parent="leg2_coxa" child="leg2_femur" />
 				<m_femur_link name="leg2_femur"
 						origin_xyz="0 0.0385 0" origin_rpy="0 3.14159 0"
 						inertia_origin_xyz="0 0.0385 0"/>
 					<m_joint name="leg2_femur__leg2_tibia" type="revolute" axis_xyz="1 0 0"
-					 effort="10000.0" lower="-1.5708" upper="1.5708" velocity="100"
-					 origin_xyz="0 0.077 0" origin_rpy="0 0 0"
-					 parent="leg2_femur" child="leg2_tibia" damping="0.7"/>
+					 effort="2.8" lower="-1.5708" upper="1.5708" velocity="5.6548668"
+					 origin_xyz="0 0.077 0" origin_rpy="0 0 0"
+					 parent="leg2_femur" child="leg2_tibia" />
 					<m_tibia_link name="leg2_tibia"
 							origin_xyz="0 0 0" origin_rpy="3.14159 0 1.5708"
@@ -65,20 +65,20 @@
 		<!-- LEG 3 (East) -->
 			<m_joint name="base_link__leg3_coxa" type="revolute" axis_xyz="0 0 1"
-					 effort="10000.0" lower="-1.5708" upper="1.5708" velocity="100"
+					 effort="2.8" lower="-1.5708" upper="1.5708" velocity="5.6548668"
 			 		 origin_xyz="0.09850 0 0" origin_rpy="0 0 -1.5708"
-					 parent="base_link" child="leg3_coxa" damping="0.7"/>
+					 parent="base_link" child="leg3_coxa" />
 			<m_coxa_link name="leg3_coxa" inertia_origin_xyz="0 0.023937 0.021"
 					origin_xyz="0 0 0.021" origin_rpy="0 0 0"/>
 				<m_joint name="leg3_coxa__leg3_femur" type="revolute" axis_xyz="1 0 0"
-						 effort="10000.0" lower="-1.5708" upper="1.5708" velocity="100"
+						 effort="2.8" lower="-1.5708" upper="1.5708" velocity="5.6548668"
 						 origin_xyz="0 0.047868 0.021" origin_rpy="0 0 0"
-						 parent="leg3_coxa" child="leg3_femur" damping="0.7"/>
+						 parent="leg3_coxa" child="leg3_femur" />
 				<m_femur_link name="leg3_femur"
 						origin_xyz="0 0.0385 0" origin_rpy="0 3.14159 0"
 						inertia_origin_xyz="0 0.0385 0"/>
 					<m_joint name="leg3_femur__leg3_tibia" type="revolute" axis_xyz="1 0 0"
-					 effort="10000.0" lower="-1.5708" upper="1.5708" velocity="100"
-					 origin_xyz="0 0.077 0" origin_rpy="0 0 0"
-					 parent="leg3_femur" child="leg3_tibia" damping="0.7"/>
+					 effort="2.8" lower="-1.5708" upper="1.5708" velocity="5.6548668"
+					 origin_xyz="0 0.077 0" origin_rpy="0 0 0"
+					 parent="leg3_femur" child="leg3_tibia" />
 					<m_tibia_link name="leg3_tibia"
 							origin_xyz="0 0 0" origin_rpy="3.14159 0 1.5708"
@@ -91,20 +91,20 @@
 		<!-- LEG 4 (West) -->
 			<m_joint name="base_link__leg4_coxa" type="revolute" axis_xyz="0 0 1"
-					 effort="10000.0" lower="-1.5708" upper="1.5708" velocity="100"
+					 effort="2.8" lower="-1.5708" upper="1.5708" velocity="5.6548668"
 			 		 origin_xyz="-0.09850 0 0" origin_rpy="0 0 1.5708"
-					 parent="base_link" child="leg4_coxa" damping="0.7"/>
+					 parent="base_link" child="leg4_coxa" />
 			<m_coxa_link name="leg4_coxa"
 					origin_xyz="0 0 0.021" origin_rpy="0 0 0" inertia_origin_xyz="0 0.023937 0.021"/>
 				<m_joint name="leg4_coxa__leg4_femur" type="revolute" axis_xyz="1 0 0"
-				 effort="10000.0" lower="-1.5708" upper="1.5708" velocity="100"
+				 effort="2.8" lower="-1.5708" upper="1.5708" velocity="5.6548668"
 				 origin_xyz="0 0.047868 0.021" origin_rpy="0 0 0"
-				 parent="leg4_coxa" child="leg4_femur" damping="0.7"/>
+				 parent="leg4_coxa" child="leg4_femur" />
 				<m_femur_link name="leg4_femur"
 						origin_xyz="0 0.0385 0" origin_rpy="0 3.14159 0"
 						inertia_origin_xyz="0 0.0385 0"/>
 					<m_joint name="leg4_femur__leg4_tibia" type="revolute" axis_xyz="1 0 0"
-					 effort="10000.0" lower="-1.5708" upper="1.5708" velocity="100"
-					 origin_xyz="0 0.077 0" origin_rpy="0 0 0"
-					 parent="leg4_femur" child="leg4_tibia" damping="0.7"/>
+					 effort="2.8" lower="-1.5708" upper="1.5708" velocity="5.6548668"
+					 origin_xyz="0 0.077 0" origin_rpy="0 0 0"
+					 parent="leg4_femur" child="leg4_tibia" />
 					<m_tibia_link name="leg4_tibia"
 							origin_xyz="0 0 0" origin_rpy="3.14159 0 1.5708"
@@ -117,20 +117,20 @@
 		<!-- LEG 5 (South East) -->
 			<m_joint name="base_link__leg5_coxa" type="revolute" axis_xyz="0 0 1"
-					 effort="10000.0" lower="-1.5708" upper="1.5708" velocity="100"
+					 effort="2.8" lower="-1.5708" upper="1.5708" velocity="5.6548668"
 			 		 origin_xyz="0.072981 -0.109608 0" origin_rpy="0 0 -2.3562"
-					 parent="base_link" child="leg5_coxa" damping="0.7"/>
+					 parent="base_link" child="leg5_coxa" />
 			<m_coxa_link name="leg5_coxa"
 					origin_xyz="0 0 0.021" origin_rpy="0 0 0" inertia_origin_xyz="0 0.023937 0.021"/>
 				<m_joint name="leg5_coxa__leg5_femur" type="revolute" axis_xyz="1 0 0"
-						 effort="10000.0" lower="-1.5708" upper="1.5708" velocity="100"
+						 effort="2.8" lower="-1.5708" upper="1.5708" velocity="5.6548668"
 						 origin_xyz="0 0.047868 0.021" origin_rpy="0 0 0"
-						 parent="leg5_coxa" child="leg5_femur" damping="0.7"/>
+						 parent="leg5_coxa" child="leg5_femur" />
 				<m_femur_link name="leg5_femur"
 						origin_xyz="0 0.0385 0" origin_rpy="0 3.14159 0"
 						inertia_origin_xyz="0 0.0385 0"/>
 					<m_joint name="leg5_femur__leg5_tibia" type="revolute" axis_xyz="1 0 0"
-					 effort="10000.0" lower="-1.5708" upper="1.5708" velocity="100"
-					 origin_xyz="0 0.077 0" origin_rpy="0 0 0"
-					 parent="leg5_femur" child="leg5_tibia" damping="0.7"/>
+					 effort="2.8" lower="-1.5708" upper="1.5708" velocity="5.6548668"
+					 origin_xyz="0 0.077 0" origin_rpy="0 0 0"
+					 parent="leg5_femur" child="leg5_tibia" />
 					<m_tibia_link name="leg5_tibia"
 							origin_xyz="0 0 0" origin_rpy="3.14159 0 1.5708"
@@ -143,20 +143,20 @@
 		<!-- LEG 6 (South West) -->
 			<m_joint name="base_link__leg6_coxa" type="revolute" axis_xyz="0 0 1"
-					 effort="10000.0" lower="-1.5708" upper="1.5708" velocity="100"
+					 effort="2.8" lower="-1.5708" upper="1.5708" velocity="5.6548668"
 			 		 origin_xyz="-0.072981 -0.109608 0" origin_rpy="0 0 2.3562"
-					 parent="base_link" child="leg6_coxa" damping="0.7"/>
+					 parent="base_link" child="leg6_coxa" />
 			<m_coxa_link name="leg6_coxa"
 					origin_xyz="0 0 0.021" origin_rpy="0 0 0" inertia_origin_xyz="0 0.023937 0.021"/>
 				<m_joint name="leg6_coxa__leg6_femur" type="revolute" axis_xyz="1 0 0"
-						 effort="10000.0" lower="-1.5708" upper="1.5708" velocity="100"
+						 effort="2.8" lower="-1.5708" upper="1.5708" velocity="5.6548668"
 						 origin_xyz="0 0.047868 0.021" origin_rpy="0 0 0"
-						 parent="leg6_coxa" child="leg6_femur" damping="0.7"/>
+						 parent="leg6_coxa" child="leg6_femur" />
 				<m_femur_link name="leg6_femur"
 						origin_xyz="0 0.0385 0" origin_rpy="0 3.14159 0"
 						inertia_origin_xyz="0 0.0385 0"/>
 					<m_joint name="leg6_femur__leg6_tibia" type="revolute" axis_xyz="1 0 0"
-					 effort="10000.0" lower="-1.5708" upper="1.5708" velocity="100"
-					 origin_xyz="0 0.077 0" origin_rpy="0 0 0"
-					 parent="leg6_femur" child="leg6_tibia" damping="0.7"/>
+					 effort="2.8" lower="-1.5708" upper="1.5708" velocity="5.6548668"
+					 origin_xyz="0 0.077 0" origin_rpy="0 0 0"
+					 parent="leg6_femur" child="leg6_tibia" />
 					<m_tibia_link name="leg6_tibia"
 							origin_xyz="0 0 0" origin_rpy="3.14159 0 1.5708"

File: hexapod_description/urdf/links_joints_macro.xacro (robot description, xacro)
@@ -125,5 +125,5 @@
 		</link>
 	</xacro:macro>
-	<xacro:macro name="m_joint" params="name type axis_xyz effort lower upper velocity origin_xyz origin_rpy parent child damping" >
+	<xacro:macro name="m_joint" params="name type axis_xyz effort lower upper velocity origin_xyz origin_rpy parent child" >
 		<joint name="${name}" type="${type}">
 			<axis xyz="${axis_xyz}" />
@@ -132,5 +132,4 @@
 			<parent link="${parent}" />
 			<child link="${child}" />
-			<dynamics damping="${damping}"/>
 		</joint>
 	</xacro:macro>
