Commit message: Added selfCollide

File: hexapod_description/urdf/links_joints_macro.xacro (robot description, xacro)
@@ -71,7 +71,7 @@
       			<origin xyz="${inertia_origin_xyz}" rpy="0 0 0"/>
       			<mass value="0.12"/>
-      			<inertia ixx="1.005e-4"			ixy="0"				ixz="0"
-      					 iyx="0"  				iyy="2.532e-5"		iyz="0"
-      					 izx="0"				izy="0"				izz="1.071e-4"/>
+      			<inertia ixx="1.005e-3"			ixy="0"				ixz="0"
+      					 iyx="0"  				iyy="2.532e-4"		iyz="0"
+      					 izx="0"				izy="0"				izz="1.071e-3"/>
     		</inertial>
 		</link>

Commit message: With the keyboard interface

File: hexapod_description/urdf/links_joints_macro.xacro (robot description, xacro)
@@ -90,5 +90,5 @@
 					<mesh filename="package://hexapod_description/meshes/leg_tibia.stl" scale="0.001 0.001 0.001" />
 				</geometry>
-				<material name="red" />
+				<material name="blue" />
 			</visual>
 			<inertial>
@@ -114,5 +114,5 @@
 					<mesh filename="package://hexapod_description/meshes/leg_rubber_tip.stl" scale="0.001 0.001 0.001" />
 				</geometry>
-				<material name="red" />
+				<material name="black" />
 			</visual>
 			<inertial>

Commit message: Cleaned the code

File: hexapod_description/urdf/links_joints_macro.xacro (robot description, xacro)
@@ -90,5 +90,5 @@
 					<mesh filename="package://hexapod_description/meshes/leg_tibia.stl" scale="0.001 0.001 0.001" />
 				</geometry>
-				<material name="blue" />
+				<material name="red" />
 			</visual>
 			<inertial>
